File: pcb/carrier/carrier.kicad_sch (KiCad schematic)
At the start: 26 parts, among them J1 Freeze footswitch, J2 Clear footswitch, J3 In (mono; grounded when empty), J4 Out L / Mono, J5 Out R (ring switch = plug det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, SW1 Single / Multi, SW2 +5 up / down, U1 Daisy Seed3

Commit message: Enclosure: 2.5 mm top panel for stocked 20 mm pots
The 25 mm RV09AF-40 shaft isn't stocked by US distributors, so the BOM
now calls for the 20 mm part (Mouser, Jameco, Tayda). The toggles fix the
board 10.39 mm under the panel, so the only way to keep shaft above the
panel is a thinner panel: 3.5 -> 2.5 mm gives 7.1 mm of shaft. Toggle
thread above panel rises to 6.4 mm, LED spacer shortens to 4 mm,
footswitch clearance rises to about 29 mm. Gerbers are unchanged
(the ordered boards still fit). STLs regenerated; all panel holes probe clear.

Co-Authored-By: Claude Opus 5.5 <noreply@anthropic.com>
Claude-Session: https://claude.ai/code/session_01JAavHVgiwWaG4iqEz4KA1Q
Parts:
- RV1, RV2, RV3, RV4, RV5, RV6, RV7: MPN Alpha RV09AF-40-25K-B10K (25 mm knurled shaft) -> Alpha RV09AF-40-20K-B10K (20 mm knurled shaft)
Changed lines of the file:
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@@
     (property "Footprint" "carrier:Potentiometer_Alpha_RV09AF-40_Vertical" (at 50 40 0) (effects (font (size 1.27 1.27)) hide))
     (property "Datasheet" "" (at 50 40 0) (effects (font (size 1.27 1.27)) hide))
-    (property "MPN" "Alpha RV09AF-40-25K-B10K (25 mm knurled shaft)" (at 50 40 0) (effects (font (size 1.27 1.27)) hide))
+    (property "MPN" "Alpha RV09AF-40-20K-B10K (20 mm knurled shaft)" (at 50 40 0) (effects (font (size 1.27 1.27)) hide))
     (pin "1")
     (pin "2")
@@
     (property "Footprint" "carrier:Potentiometer_Alpha_RV09AF-40_Vertical" (at 50 70 0) (effects (font (size 1.27 1.27)) hide))
     (property "Datasheet" "" (at 50 70 0) (effects (font (size 1.27 1.27)) hide))
-    (property "MPN" "Alpha RV09AF-40-25K-B10K (25 mm knurled shaft)" (at 50 70 0) (effects (font (size 1.27 1.27)) hide))
+    (property "MPN" "Alpha RV09AF-40-20K-B10K (20 mm knurled shaft)" (at 50 70 0) (effects (font (size 1.27 1.27)) hide))
     (pin "1")
     (pin "2")
@@
     (property "Footprint" "carrier:Potentiometer_Alpha_RV09AF-40_Vertical" (at 50 100 0) (effects (font (size 1.27 1.27)) hide))
     (property "Datasheet" "" (at 50 100 0) (effects (font (size 1.27 1.27)) hide))
-    (property "MPN" "Alpha RV09AF-40-25K-B10K (25 mm knurled shaft)" (at 50 100 0) (effects (font (size 1.27 1.27)) hide))
+    (property "MPN" "Alpha RV09AF-40-20K-B10K (20 mm knurled shaft)" (at 50 100 0) (effects (font (size 1.27 1.27)) hide))
     (pin "1")
     (pin "2")
@@
     (property "Footprint" "carrier:Potentiometer_Alpha_RV09AF-40_Vertical" (at 50 130 0) (effects (font (size 1.27 1.27)) hide))
     (property "Datasheet" "" (at 50 130 0) (effects (font (size 1.27 1.27)) hide))
-    (property "MPN" "Alpha RV09AF-40-25K-B10K (25 mm knurled shaft)" (at 50 130 0) (effects (font (size 1.27 1.27)) hide))
+    (property "MPN" "Alpha RV09AF-40-20K-B10K (20 mm knurled shaft)" (at 50 130 0) (effects (font (size 1.27 1.27)) hide))
     (pin "1")
     (pin "2")
@@
     (property "Footprint" "carrier:Potentiometer_Alpha_RV09AF-40_Vertical" (at 50 160 0) (effects (font (size 1.27 1.27)) hide))
     (property "Datasheet" "" (at 50 160 0) (effects (font (size 1.27 1.27)) hide))
-    (property "MPN" "Alpha RV09AF-40-25K-B10K (25 mm knurled shaft)" (at 50 160 0) (effects (font (size 1.27 1.27)) hide))
+    (property "MPN" "Alpha RV09AF-40-20K-B10K (20 mm knurled shaft)" (at 50 160 0) (effects (font (size 1.27 1.27)) hide))
     (pin "1")
     (pin "2")
@@
     (property "Footprint" "carrier:Potentiometer_Alpha_RV09AF-40_Vertical" (at 50 190 0) (effects (font (size 1.27 1.27)) hide))
     (property "Datasheet" "" (at 50 190 0) (effects (font (size 1.27 1.27)) hide))
-    (property "MPN" "Alpha RV09AF-40-25K-B10K (25 mm knurled shaft)" (at 50 190 0) (effects (font (size 1.27 1.27)) hide))
+    (property "MPN" "Alpha RV09AF-40-20K-B10K (20 mm knurled shaft)" (at 50 190 0) (effects (font (size 1.27 1.27)) hide))
     (pin "1")
     (pin "2")
@@
     (property "Footprint" "carrier:Potentiometer_Alpha_RV09AF-40_Vertical" (at 50 220 0) (effects (font (size 1.27 1.27)) hide))
     (property "Datasheet" "" (at 50 220 0) (effects (font (size 1.27 1.27)) hide))
-    (property "MPN" "Alpha RV09AF-40-25K-B10K (25 mm knurled shaft)" (at 50 220 0) (effects (font (size 1.27 1.27)) hide))
+    (property "MPN" "Alpha RV09AF-40-20K-B10K (20 mm knurled shaft)" (at 50 220 0) (effects (font (size 1.27 1.27)) hide))
     (pin "1")
     (pin "2")

Commit message: BOM: Digi-Key-friendly toggle (with nuts) and capacitor, 4 mm LED spacer
Co-Authored-By: Claude Opus 5.5 <noreply@anthropic.com>
Claude-Session: https://claude.ai/code/session_01JAavHVgiwWaG4iqEz4KA1Q
Parts:
- C1, C2: MPN 10 uF 25 V X7R radial MLCC, 5.08 mm leads (e.g. TDK FG28X7R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 -> 10 uF ≥25 V X7R radial MLCC, 5.08 mm leads (e.g. TDK FG20X7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
- D1: MPN 5 mm bi-colour LED, common cathode (red/green), on a 5 mm s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 -> 5 mm bi-colour LED, common cathode (red/green), on a 4 mm s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
- SW1, SW2: MPN E-Switch 100SP1T1B1M2QE -> E-Switch 100SP1T1B1M2QEH (H = with nuts; 100SP1T1B1M2QE wit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
Changed lines of the file:
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@@
     (property "Footprint" "Capacitor_THT:C_Disc_D5.0mm_W2.5mm_P5.00mm" (at 395 95 0) (effects (font (size 1.27 1.27)) hide))
     (property "Datasheet" "" (at 395 95 0) (effects (font (size 1.27 1.27)) hide))
-    (property "MPN" "10 uF 25 V X7R radial MLCC, 5.08 mm leads (e.g. TDK FG28X7R1E106KRT06)" (at 395 95 0) (effects (font (size 1.27 1.27)) hide))
+    (property "MPN" "10 uF ≥25 V X7R radial MLCC, 5.08 mm leads (e.g. TDK FG20X7R1H106KRT06, 50 V, on Digi-Key)" (at 395 95 0) (effects (font (size 1.27 1.27)) hide))
     (pin "1")
     (pin "2")
@@
     (property "Footprint" "Capacitor_THT:C_Disc_D5.0mm_W2.5mm_P5.00mm" (at 395 145 0) (effects (font (size 1.27 1.27)) hide))
     (property "Datasheet" "" (at 395 145 0) (effects (font (size 1.27 1.27)) hide))
-    (property "MPN" "10 uF 25 V X7R radial MLCC, 5.08 mm leads (e.g. TDK FG28X7R1E106KRT06)" (at 395 145 0) (effects (font (size 1.27 1.27)) hide))
+    (property "MPN" "10 uF ≥25 V X7R radial MLCC, 5.08 mm leads (e.g. TDK FG20X7R1H106KRT06, 50 V, on Digi-Key)" (at 395 145 0) (effects (font (size 1.27 1.27)) hide))
     (pin "1")
     (pin "2")
@@
     (property "Footprint" "carrier:SW_E-Switch_100SP_M2_PCB" (at 300 225 0) (effects (font (size 1.27 1.27)) hide))
     (property "Datasheet" "" (at 300 225 0) (effects (font (size 1.27 1.27)) hide))
-    (property "MPN" "E-Switch 100SP1T1B1M2QE" (at 300 225 0) (effects (font (size 1.27 1.27)) hide))
+    (property "MPN" "E-Switch 100SP1T1B1M2QEH (H = with nuts; 100SP1T1B1M2QE without)" (at 300 225 0) (effects (font (size 1.27 1.27)) hide))
     (pin "1")
     (pin "2")
@@
     (property "Footprint" "carrier:SW_E-Switch_100SP_M2_PCB" (at 350 225 0) (effects (font (size 1.27 1.27)) hide))
     (property "Datasheet" "" (at 350 225 0) (effects (font (size 1.27 1.27)) hide))
-    (property "MPN" "E-Switch 100SP1T1B1M2QE" (at 350 225 0) (effects (font (size 1.27 1.27)) hide))
+    (property "MPN" "E-Switch 100SP1T1B1M2QEH (H = with nuts; 100SP1T1B1M2QE without)" (at 350 225 0) (effects (font (size 1.27 1.27)) hide))
     (pin "1")
     (pin "2")
@@
     (property "Footprint" "LED_THT:LED_D5.0mm-3" (at 230 245 0) (effects (font (size 1.27 1.27)) hide))
     (property "Datasheet" "" (at 230 245 0) (effects (font (size 1.27 1.27)) hide))
-    (property "MPN" "5 mm bi-colour LED, common cathode (red/green), on a 5 mm spacer" (at 230 245 0) (effects (font (size 1.27 1.27)) hide))
+    (property "MPN" "5 mm bi-colour LED, common cathode (red/green), on a 4 mm spacer" (at 230 245 0) (effects (font (size 1.27 1.27)) hide))
     (pin "1")
     (pin "2")

Commit message: BOM: gold-contact toggle 100SP1T1B1M2RE (same body and pins)
Co-Authored-By: Claude Opus 5.5 <noreply@anthropic.com>
Claude-Session: https://claude.ai/code/session_01JAavHVgiwWaG4iqEz4KA1Q
Parts:
- SW1, SW2: MPN E-Switch 100SP1T1B1M2QEH (H = with nuts; 100SP1T1B1M2QE wit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 -> E-Switch 100SP1T1B1M2RE (gold contacts; any 100SP1…M2 fits)
Changed lines of the file:
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@@
     (property "Footprint" "carrier:SW_E-Switch_100SP_M2_PCB" (at 300 225 0) (effects (font (size 1.27 1.27)) hide))
     (property "Datasheet" "" (at 300 225 0) (effects (font (size 1.27 1.27)) hide))
-    (property "MPN" "E-Switch 100SP1T1B1M2QEH (H = with nuts; 100SP1T1B1M2QE without)" (at 300 225 0) (effects (font (size 1.27 1.27)) hide))
+    (property "MPN" "E-Switch 100SP1T1B1M2RE (gold contacts; any 100SP1…M2 fits)" (at 300 225 0) (effects (font (size 1.27 1.27)) hide))
     (pin "1")
     (pin "2")
@@
     (property "Footprint" "carrier:SW_E-Switch_100SP_M2_PCB" (at 350 225 0) (effects (font (size 1.27 1.27)) hide))
     (property "Datasheet" "" (at 350 225 0) (effects (font (size 1.27 1.27)) hide))
-    (property "MPN" "E-Switch 100SP1T1B1M2QEH (H = with nuts; 100SP1T1B1M2QE without)" (at 350 225 0) (effects (font (size 1.27 1.27)) hide))
+    (property "MPN" "E-Switch 100SP1T1B1M2RE (gold contacts; any 100SP1…M2 fits)" (at 350 225 0) (effects (font (size 1.27 1.27)) hide))
     (pin "1")
     (pin "2")

Commit message: Drop JST connectors: footswitch leads solder straight into J1/J2
Co-Authored-By: Claude Opus 5.5 <noreply@anthropic.com>
Claude-Session: https://claude.ai/code/session_01JAavHVgiwWaG4iqEz4KA1Q
Parts:
- J1, J2: MPN JST B2B-PH-K; footswitch: soft-touch momentary SPST, panel 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 -> No connector: solder 24-26 AWG leads into the J pads (eithe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
Changed lines of the file:
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@@
   (title_block (title "Daisy Freeze Pedal - carrier board") (date "2026-10-26") (rev "A")
     (comment 1 "Generated by gen_schematic.py from one netlist definition - edit the script, not the sheet")
-    (comment 2 "Bare board, all through-hole. Pots/toggles/LED on top; Seed3 + jacks underneath; footswitches on JST PH")
+    (comment 2 "Bare board, all through-hole. Pots/toggles/LED on top; Seed3 + jacks underneath; footswitches wired to J1/J2")
     (comment 3 "One carrier ground: Seed AGND (pin 20) and DGND (pin 40) both tie to the GND pour"))
   (symbol (lib_id "carrier:DaisySeed") (at 210 150 0) (unit 1)
@@
     (property "Footprint" "Connector_JST:JST_PH_B2B-PH-K_1x02_P2.00mm_Vertical" (at 140 225 0) (effects (font (size 1.27 1.27)) hide))
     (property "Datasheet" "" (at 140 225 0) (effects (font (size 1.27 1.27)) hide))
-    (property "MPN" "JST B2B-PH-K; footswitch: soft-touch momentary SPST, panel mounted" (at 140 225 0) (effects (font (size 1.27 1.27)) hide))
+    (property "MPN" "No connector: solder 24-26 AWG leads into the J pads (either way round). Footswitch: soft-touch momentary SPST, panel mounted (Tayda)" (at 140 225 0) (effects (font (size 1.27 1.27)) hide))
     (pin "1")
     (pin "2")
@@
     (property "Footprint" "Connector_JST:JST_PH_B2B-PH-K_1x02_P2.00mm_Vertical" (at 140 250 0) (effects (font (size 1.27 1.27)) hide))
     (property "Datasheet" "" (at 140 250 0) (effects (font (size 1.27 1.27)) hide))
-    (property "MPN" "JST B2B-PH-K; footswitch: soft-touch momentary SPST, panel mounted" (at 140 250 0) (effects (font (size 1.27 1.27)) hide))
-    (pin "1")
-    (pin "2")
+    (property "MPN" "No connector: solder 24-26 AWG leads into the J pads (either way round). Footswitch: soft-touch momentary SPST, panel mounted (Tayda)" (at 140 250 0) (effects (font (size 1.27 1.27)) hide))
+    (pin "1")
+    (pin "2")
